File: MagnavoxOdyssey1/J9_Vert_Sync_Generator.sch (KiCad schematic (older format))
At the start: 15 parts

Commit message: mais outro pedação do circuito transcrito :-)
Parts:
- removed 10_C3, 10_C4: 10 MFD 25V, symbol CAPAPOL
- removed 10_L1: 620UH, symbol INDUCTOR
- 9_C1: renamed from 10_C1; value 470 -> .1
- 9_C2: renamed from 10_C2; value 680 -> .1
- 9_Q1: renamed from 10_Q1; value 142N7 -> 142N9
- 9_Q2: renamed from 10_Q2; value 134P5 -> 134P1
- 9_R1: renamed from 10_R1; value 1k -> 2.2k
- 9_R2: renamed from 10_R2; value 150k 5% -> 180k 5%
- 9_R3: renamed from 10_R3; value 820 -> 470
- 9_R4: renamed from 10_R4; value 3.3k 5% -> 820
- 9_R6: renamed from 10_R6; value 1k -> 2.2k
- renumbered 10_Q3 to 9_Q3, 10_R5 to 9_R5, 10_R7 to 9_R7
Connections:
- net (9)_5.6V: now reaches 9_Q2.1 (E), 9_Q3.3 (C), 9_R1.2
- net (3)_HORIZ_RATE renamed (3)_VERT_RATE
- net (7)_HSYNC renamed (7)_VERT_IN
Other:
- note added: "703492-3"
- note added: "VERT SYNC GENERATOR"
- note removed: "703491-3"
- note removed: "HORIZ SYNC GENERATOR"
- moved on the sheet: 9_R1
Changed lines of the file:
@@
 LIBS:valves
 LIBS:ferrite
+LIBS:conn_22x2
 LIBS:MagnavoxOdyssey1-cache
 EELAYER 25 0
@@
 $Descr A4 11693 8268
 encoding utf-8
-Sheet 5 5
+Sheet 6 7
 Title ""
 Date ""
@@
 $EndDescr
 $Comp
-L NPN 10_Q1
+L NPN 9_Q1
 U 1 1 588F195D
 P 4250 4300
-F 0 "10_Q1" H 4440 4346 50  0000 L CNN
-F 1 "142N7" H 4440 4255 50  0000 L CNN
+F 0 "9_Q1" H 4440 4346 50  0000 L CNN
+F 1 "142N9" H 4440 4255 50  0000 L CNN
 F 2 "" H 4250 4300 60  0000 C CNN
 F 3 "" H 4250 4300 60  0000 C CNN
@@
 $EndComp
 $Comp
-L NPN 10_Q3
+L NPN 9_Q3
 U 1 1 588F19A5
 P 7900 4100
-F 0 "10_Q3" H 8091 4146 50  0000 L CNN
+F 0 "9_Q3" H 8091 4146 50  0000 L CNN
 F 1 "142N9" H 8091 4055 50  0000 L CNN
 F 2 "" H 7900 4100 60  0000 C CNN
@@
 $EndComp
 $Comp
-L PNP 10_Q2
+L PNP 9_Q2
 U 1 1 588F19E5
 P 7350 3800
-F 0 "10_Q2" H 7541 3747 60  0000 L CNN
-F 1 "134P5" H 7541 3853 60  0000 L CNN
+F 0 "9_Q2" H 7541 3747 60  0000 L CNN
+F 1 "134P1" H 7541 3853 60  0000 L CNN
 F 2 "" H 7350 3800 60  0000 C CNN
 F 3 "" H 7350 3800 60  0000 C CNN
@@
 $EndComp
 $Comp
-L CP1 10_C1
+L CP1 9_C1
 U 1 1 588F1A19
 P 5450 4300
-F 0 "10_C1" V 5720 4300 50  0000 C CNN
-F 1 "470" V 5629 4300 50  0000 C CNN
+F 0 "9_C1" V 5720 4300 50  0000 C CNN
+F 1 ".1" V 5629 4300 50  0000 C CNN
 F 2 "" H 5450 4300 60  0000 C CNN
 F 3 "" H 5450 4300 60  0000 C CNN
@@
 $EndComp
 $Comp
-L R 10_R4
+L R 9_R4
 U 1 1 588F1AE3
 P 6200 4300
-F 0 "10_R4" V 6015 4300 40  0000 C CNN
-F 1 "3.3k 5%" V 6091 4300 40  0000 C CNN
+F 0 "9_R4" V 6015 4300 40  0000 C CNN
+F 1 "820" V 6091 4300 40  0000 C CNN
 F 2 "" V 6130 4300 30  0000 C CNN
 F 3 "" H 6200 4300 30  0000 C CNN
@@
 $EndComp
 $Comp
-L R 10_R2
+L R 9_R2
 U 1 1 588F1B69
 P 4850 4750
-F 0 "10_R2" H 4779 4712 40  0000 R CNN
-F 1 "150k 5%" H 4779 4788 40  0000 R CNN
+F 0 "9_R2" H 4779 4712 40  0000 R CNN
+F 1 "180k 5%" H 4779 4788 40  0000 R CNN
 F 2 "" V 4780 4750 30  0000 C CNN
 F 3 "" H 4850 4750 30  0000 C CNN
@@
 $EndComp
 $Comp
-L R 10_R5
+L R 9_R5
 U 1 1 588F1BE1
 P 6800 4700
-F 0 "10_R5" H 6729 4662 40  0000 R CNN
+F 0 "9_R5" H 6729 4662 40  0000 R CNN
 F 1 "300k 5%" H 6729 4738 40  0000 R CNN
 F 2 "" V 6730 4700 30  0000 C CNN
@@
 $EndComp
 $Comp
-L R 10_R3
+L R 9_R3
 U 1 1 588F1C71
 P 5450 3800
-F 0 "10_R3" V 5265 3800 40  0000 C CNN
-F 1 "820" V 5341 3800 40  0000 C CNN
+F 0 "9_R3" V 5265 3800 40  0000 C CNN
+F 1 "470" V 5341 3800 40  0000 C CNN
 F 2 "" V 5380 3800 30  0000 C CNN
 F 3 "" H 5450 3800 30  0000 C CNN
@@
 $EndComp
 $Comp
-L CP1 10_C2
+L CP1 9_C2
 U 1 1 588F1CB5
 P 6200 3800
-F 0 "10_C2" V 6470 3800 50  0000 C CNN
-F 1 "680" V 6379 3800 50  0000 C CNN
+F 0 "9_C2" V 6470 3800 50  0000 C CNN
+F 1 ".1" V 6379 3800 50  0000 C CNN
 F 2 "" H 6200 3800 60  0000 C CNN
 F 3 "" H 6200 3800 60  0000 C CNN
@@
 $EndComp
 $Comp
-L R 10_R1
+L R 9_R1
 U 1 1 588F1D79
-P 4850 3400
-F 0 "10_R1" H 4779 3362 40  0000 R CNN
-F 1 "1k" H 4779 3438 40  0000 R CNN
-F 2 "" V 4780 3400 30  0000 C CNN
-F 3 "" H 4850 3400 30  0000 C CNN
-	1    4850 3400
-	-1   0    0    1
-$EndComp
-$Comp
-L R 10_R6
+P 4150 3400
+F 0 "9_R1" H 4079 3362 40  0000 R CNN
+F 1 "2.2k" H 4079 3438 40  0000 R CNN
+F 2 "" V 4080 3400 30  0000 C CNN
+F 3 "" H 4150 3400 30  0000 C CNN
+	1    4150 3400
+	-1   0    0    1
+$EndComp
+$Comp
+L R 9_R6
 U 1 1 588F1F59
 P 7450 4700
-F 0 "10_R6" H 7379 4662 40  0000 R CNN
-F 1 "1k" H 7379 4738 40  0000 R CNN
+F 0 "9_R6" H 7379 4662 40  0000 R CNN
+F 1 "2.2k" H 7379 4738 40  0000 R CNN
 F 2 "" V 7380 4700 30  0000 C CNN
 F 3 "" H 7450 4700 30  0000 C CNN
@@
 $EndComp
 $Comp
-L R 10_R7
+L R 9_R7
 U 1 1 588F1FC4
 P 8000 4700
-F 0 "10_R7" H 7929 4662 40  0000 R CNN
+F 0 "9_R7" H 7929 4662 40  0000 R CNN
 F 1 "470" H 7929 4738 40  0000 R CNN
 F 2 "" V 7930 4700 30  0000 C CNN
@@
 	6000 3800 5700 3800
 Wire Wire Line
-	4150 3800 4150 4100
+	4150 3650 4150 4100
 Wire Wire Line
 	3000 3800 5200 3800
-Wire Wire Line
-	4850 3650 4850 3800
-Connection ~ 4850 3800
-Wire Wire Line
-	4850 3000 4850 3150
-Wire Wire Line
-	4150 3000 8000 3000
+Connection ~ 4150 3800
+Wire Wire Line
+	4150 3000 4150 3150
 Wire Wire Line
 	7450 3000 7450 3600
@@
 	8000 5050 8000 4950
 $Comp
-L GND #PWR024
+L GND #PWR033
 U 1 1 588F20E4
 P 7450 5200
-F 0 "#PWR024" H 7450 5200 30  0001 C CNN
+F 0 "#PWR033" H 7450 5200 30  0001 C CNN
 F 1 "GND" H 7450 5130 30  0001 C CNN
 F 2 "" H 7450 5200 60  0001 C CNN
@@
 $EndComp
 $Comp
-L GND #PWR025
+L GND #PWR034
 U 1 1 588F211A
 P 6800 5200
-F 0 "#PWR025" H 6800 5200 30  0001 C CNN
+F 0 "#PWR034" H 6800 5200 30  0001 C CNN
 F 1 "GND" H 6800 5130 30  0001 C CNN
 F 2 "" H 6800 5200 60  0001 C CNN
@@
 	6800 4950 6800 5200
 $Comp
-L GND #PWR026
+L GND #PWR035
 U 1 1 588F2289
 P 4150 4700
-F 0 "#PWR026" H 4150 4700 30  0001 C CNN
+F 0 "#PWR035" H 4150 4700 30  0001 C CNN
 F 1 "GND" H 4150 4630 30  0001 C CNN
 F 2 "" H 4150 4700 60  0001 C CNN
@@
 Wire Wire Line
 	4150 4500 4150 4700
-Text HLabel 3000 3800 0    60   Input ~ 0
-(3)_HORIZ_RATE
-Connection ~ 4150 3800
+Text HLabel 3000 3800 0    60   Output ~ 0
+(3)_VERT_RATE
 Text HLabel 8600 4400 2    60   Output ~ 0
-(7)_HSYNC
+(7)_VERT_IN
 Wire Wire Line
 	8600 4400 8000 4400
@@
 (5)
 $Comp
-L GND #PWR027
+L GND #PWR036
 U 1 1 588F26A8
 P 8450 5200
-F 0 "#PWR027" H 8450 5200 30  0001 C CNN
+F 0 "#PWR036" H 8450 5200 30  0001 C CNN
 F 1 "GND" H 8450 5130 30  0001 C CNN
 F 2 "" H 8450 5200 60  0001 C CNN
@@
 	4850 5200 3000 5200
 Text HLabel 3000 3000 0    60   Input ~ 0
-(9)
-$Comp
-L CAPAPOL 10_C3
-U 1 1 588F2EC3
-P 3450 3350
-F 0 "10_C3" H 3559 3388 40  0000 L CNN
-F 1 "10 MFD 25V" H 3559 3312 40  0000 L CNN
-F 2 "" H 3550 3200 30  0000 C CNN
-F 3 "" H 3450 3350 300 0000 C CNN
-	1    3450 3350
-	1    0    0    -1
-$EndComp
-$Comp
-L CAPAPOL 10_C4
-U 1 1 588F2F26
-P 4300 3350
-F 0 "10_C4" H 4409 3388 40  0000 L CNN
-F 1 "10 MFD 25V" H 4409 3312 40  0000 L CNN
-F 2 "" H 4400 3200 30  0000 C CNN
-F 3 "" H 4300 3350 300 0000 C CNN
-	1    4300 3350
-	1    0    0    -1
-$EndComp
-$Comp
-L INDUCTOR 10_L1
-U 1 1 588F2F68
-P 3850 3000
-F 0 "10_L1" V 4043 3000 40  0000 C CNN
-F 1 "620UH" V 3967 3000 40  0000 C CNN
-F 2 "" H 3850 3000 60  0000 C CNN
-F 3 "" H 3850 3000 60  0000 C CNN
-	1    3850 3000
-	0    -1   -1   0
-$EndComp
-$Comp
-L GND #PWR028
-U 1 1 588F30C1
-P 4300 3650
-F 0 "#PWR028" H 4300 3650 30  0001 C CNN
-F 1 "GND" H 4300 3580 30  0001 C CNN
-F 2 "" H 4300 3650 60  0001 C CNN
-F 3 "" H 4300 3650 60  0001 C CNN
-	1    4300 3650
-	1    0    0    -1
-$EndComp
-$Comp
-L GND #PWR029
-U 1 1 588F3100
-P 3450 3650
-F 0 "#PWR029" H 3450 3650 30  0001 C CNN
-F 1 "GND" H 3450 3580 30  0001 C CNN
-F 2 "" H 3450 3650 60  0001 C CNN
-F 3 "" H 3450 3650 60  0001 C CNN
-	1    3450 3650
-	1    0    0    -1
-$EndComp
-Wire Wire Line
-	4300 3150 4300 3000
-Connection ~ 4850 3000
-Connection ~ 4300 3000
-Wire Wire Line
-	4300 3550 4300 3650
-Wire Wire Line
-	3450 3550 3450 3650
-Wire Wire Line
-	3450 3150 3450 3000
-Wire Wire Line
-	3000 3000 3550 3000
-Connection ~ 3450 3000
+(9)_5.6V
+Connection ~ 4150 3000
 Wire Notes Line
 	3000 2100 3000 5700
@@
 	8600 2100 3000 2100
 Text Notes 4450 2500 0    157  ~ 0
-HORIZ SYNC GENERATOR
+VERT SYNC GENERATOR
 Text Notes 5300 2700 0    118  ~ 0
-703491-3
+703492-3
+Wire Wire Line
+	3000 3000 8000 3000
 $EndSCHEMATC
