File: MagnavoxOdyssey1/MagnavoxOdyssey1.sch (KiCad schematic (older format))
At the start: 29 parts

Commit message: mais outro pedação do circuito transcrito :-)
Parts:
- removed R?: R, symbol R
- added GAME_CARD_1: CONN_22X2, symbol CONN_22X2
- added JU2, JU8: JUMPER, symbol JUMPER
Connections:
- net GAME_CARD_10 is gone; now on net +5.6V: R21.2
- net GAME_CARD_14 is gone; now on net +5.6V: R15.2, R18.2
- net GAME_CARD_16 is gone; now on net +5.6V: R20.1
- net +5.6V: now also GAME_CARD_1.10 (P10), GAME_CARD_1.14 (P14), GAME_CARD_1.16 (P16), GAME_CARD_1.20 (P20), GAME_CARD_1.22 (P22), GAME_CARD_1.36 (P36), GAME_CARD_1.6 (P6), GAME_CARD_1.8 (P8)
- net GAME_CARD_12: now also GAME_CARD_1.12 (P12)
- net at R39.2, R39.3: now also R23.1, TM1.1
- net J10 - HORIZ SYNC GENERATOR/(6) renamed J10 - HORIZ SYNC GENERATOR 703491-3/(6)
- net J9 - VERT SYNC GENERATOR/(6) renamed J9 - VERT SYNC GENERATOR 703492-3/(6)
- net J9 - VERT SYNC GENERATOR/(9) renamed J9 - VERT SYNC GENERATOR 703492-3/(9)_5.6V
- new net GAME_CARD_11: GAME_CARD_1.11 (P11), JU2.1
- new net GAME_CARD_17: GAME_CARD_1.17 (P17), JU8.1
- new net J16 - FLIP-FLOP/BALL 703494-2/(3): JU8.2
- new net J16 - FLIP-FLOP/BALL 703494-2/(5): JU2.2
- no-connect marks 2 -> 9
Other:
- note added: "NOTES:\nUNLESS OTHERWISE SPECIFIED\n1. CAPACITANCE VALUES 1 OR GREATER ARE IN PICOFARADS.\n2. CAPACITANCE VALUES LESS THAN 1 ARE IN MICROFARADS.\n3. RESISTORS ARE 1/4 WATT, 10%.\n4. (TRIANGLE) = ADD JUMPERS WHERE PARTS INDICATED.\n5. (ASTERISK) = SPACE PROVIDED ON LAYOUT, NO JUMPER.\n6. DIODES IN CIRCLES ARE GERMANIUM, OTHERS ARE SILICON.\n7. VOLTAGE READINGS TAKEN WITH CARD/\n UNLESS OTHERWISE N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"
- moved on the sheet: C6, R22, R23, R24, R37, R38, R39, TM1, TM2, TP2

Commit message: wip :-D
Parts:
- added C1: 220 MFD 10V, symbol CAPAPOL
- added C4: 47 MFD 16V, symbol CAPAPOL
- added R1: 1.2k, symbol R
- added R13: 33k 5%, symbol R
- added R14: 6.8k, symbol R
- added R2: 2.7k, symbol R
- added R3: 9k, symbol POT
- added R4: 15k, symbol POT
- added R5: 10k, symbol R
- added R6: 50k, symbol POT
- added R7: 27k, symbol R
- added R8: 4.7k, symbol R
- added R9: 8.2k, symbol R
Connections:
- net VERT_IN is gone; now on net GAME_CARD_29: TP2.1
- net +5.6V: now also R5.2, R7.2; no longer GAME_CARD_1.36 (P36)
- net GAME_CARD_36: now also GAME_CARD_1.36 (P36)
- net GND: now also C1.2, C4.2, R13.1
- net GAME_CARD_25: now reaches GAME_CARD_1.25 (P25)
- net GAME_CARD_29: now reaches GAME_CARD_1.29 (P29)
- net GAME_CARD_32: now reaches GAME_CARD_1.32 (P32)
- net GAME_CARD_32: now also R1.1
- net GAME_CARD_34: now reaches GAME_CARD_1.34 (P34)
- net GAME_CARD_34: now also R2.1
- net GAME_CARD_40: now reaches GAME_CARD_1.40 (P40)
- net GAME_CARD_40: now also R8.2
- net GAME_CARD_42: now reaches GAME_CARD_1.42 (P42)
- net GAME_CARD_42: now also R9.1
- net GAME_CARD_44: now reaches GAME_CARD_1.44 (P44)
- net GAME_CARD_44: now also R14.1
- new net: R6.1, R7.1
- new net: R2.2, R3.1
- new net: R4.1, R5.1
- new net J8 - BALL GENERATOR 703493-2/(2): C4.1, R14.2, R8.1, R9.2
- new net J8 - BALL GENERATOR 703493-2/(4): R4.2, R4.3
- new net J8 - BALL GENERATOR 703493-2/(7): R6.2, R6.3
- new net J8 - BALL GENERATOR 703493-2/(9): C1.1, R1.2, R13.2, R3.2, R3.3
- no-connect marks 9 -> 32
Other:
- note added: ".7V"
- note added: "1.5V TO 4.5V"
- note added: "3.2V"
- note added: "BALL\nHEIGHT"
- note added: "BALL\nSPEED"
- note added: "BALL\nWIDTH"
- moved on the sheet: C3, C5, C6, GAME_CARD_1, JU2, JU8, R10, R11, R12, R15, R17, R18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

Commit message: a lot more...
Parts:
- added C10: 4.7 MFD 50V, symbol CAPAPOL
- added C12: 100 MFD 10V, symbol CAPAPOL
- added C7, C9: 10 MFD 35V, symbol CAPAPOL
- added C8: 47 MFD 50V, symbol CAPAPOL
- added FB4: FERRITE, symbol FERRITE
- added JU12: JUMPER, symbol JUMPER
- added R26, R32: 50k, symbol POT
- added R27, R33: 27k, symbol R
- added R28, R31: 15k, symbol POT
- added R29, R30: 10k, symbol R
- added R?: 8.2k, symbol R
- added TP3: HORIZ, symbol TST
- TP2: value SWEEP INPUT -> VERT
Connections:
- net +5.6V: now also FB4.2, R27.2, R29.2, R30.2, R33.2
- net GAME_CARD_34: now also GAME_CARD_1.30 (P30)
- net GND: now also C10.2, C12.2, C7.2, C8.2, C9.2
- net HORIZ_IN: now also TP3.1
- net at GAME_CARD_1.2 (P2): now also GAME_CARD_1.4 (P4)
- net GAME_CARD_21: now reaches GAME_CARD_1.21 (P21)
- net at GAME_CARD_1.26 (P26): now also C12.1
- net at GAME_CARD_1.31 (P31): now also GAME_CARD_1.39 (P39)
- net at GAME_CARD_1.35 (P35): now also GAME_CARD_1.37 (P37)
- net W3: now reaches GAME_CARD_1.41 (P41)
- net GAME_CARD_5: now reaches GAME_CARD_1.5 (P5)
- net GAME_CARD_5: now also JU12.2
- net GAME_CARD_29 renamed VERT_IN
- new net: R26.1, R27.1
- new net: R28.1, R29.1
- new net: R32.1, R33.1
- new net: R30.1, R31.1
- new net CONTROL_1_HORIZ: C7.1
- new net CONTROL_1_VERT: R?.1
- new net CONTROL_2_HORIZ: C9.1
- new net CONTROL_2_VERT: C10.1, JU12.1
- new net J5 - PLAYER NO.2 GEN 703493-2/(4): R31.2, R31.3
- new net J5 - PLAYER NO.2 GEN 703493-2/(6): FB4.1
- new net J5 - PLAYER NO.2 GEN 703493-2/(7): R32.2, R32.3
- new net J6 - PLAYER NO.1 GEN 703493-2/(2): C8.1, R?.2
- new net J6 - PLAYER NO.1 GEN 703493-2/(4): R28.2, R28.3
- new net J6 - PLAYER NO.1 GEN 703493-2/(7): R26.2, R26.3
- no-connect marks 32 -> 21
Other:
- note added: ".1V"
- note added: ".3V"
- note added: "1.0V TO MODULATOR"
- note added: "1.8V TO 3.6V"
- note added: "3.6V"
- note added: "COMPOSITE\nVIDEO"
- note added: "PLAYER\nNO.1\nHEIGHT"
- note added: "PLAYER\nNO.1\nWIDTH"
- note added: "PLAYER\nNO.2\nHEIGHT"
- note added: "PLAYER\nNO.2\nWIDTH"
- moved on the sheet: C1, C17, C18, C3, C4, C5, C6, FB1, FB2, GAME_CARD_1, JU2, JU8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

Commit message: a bit more...
Parts:
- added C11: .001, symbol CP1
- added C16, C20: 330, symbol CP1
- added C19: 1000, symbol CP1
- added D2, D3, D4, D5, D6, D7, D8: DIODE, symbol DIODE
- added J20: CONN_6, symbol CONN_6
- added J3, J4: CONN_12, symbol CONN_12
- added Q2: 142N9, symbol NPN
- added R16, R46: 10k, symbol R
- added R44: 22k, symbol R
- added R47: 4.7k, symbol R
- added R48: 2.2k, symbol R
- added R51: 39, symbol R
- added SCR1: THYRISTOR, symbol THYRISTOR
- added Z2: 6.8V, symbol ZENER
Connections:
- net CONTROL_1_HORIZ: now also J4.11 (P11)
- net CONTROL_1_VERT: now also J4.8 (P8)
- net CONTROL_2_HORIZ: now also J3.11 (P11)
- net CONTROL_2_VERT: now also J3.8 (P8)
- net GND: now also C11.2, C16.2, C19.2, C20.2, J20.4, J3.10 (P10), J4.10 (P10), Q2.1 (E), R46.1, SCR1.K, Z2.1 (A)
- net GAME_CARD_18: now reaches GAME_CARD_1.18 (P18)
- net GAME_CARD_18: now also R47.2
- net GAME_CARD_23: now reaches GAME_CARD_1.19 (P19)
- net GAME_CARD_23: now also C11.1, J20.6, Q2.3 (C), R51.1
- net GAME_CARD_24: now reaches GAME_CARD_1.24 (P24)
- net GAME_CARD_24: now also C19.1, J20.3
- net GAME_CARD_33: now reaches GAME_CARD_1.33 (P33)
- net GAME_CARD_33: now also D4.1 (A), R47.1
- new net: C20.1, J20.1, R44.2, Z2.2 (K)
- new net: D2.2 (K), D3.2 (K), Q2.2 (B)
- new net: R16.1, R44.1, R46.2, R48.1, SCR1.G
- new net: D4.2 (K), R48.2
- new net: R51.2, SCR1.A
- new net CONTROL_1_BLK_RED: J4.12 (P12)
- new net CONTROL_1_BLU: D6.2 (K), J4.6 (P6)
- new net CONTROL_1_BRN: J4.1 (P1)
- new net CONTROL_1_ENGLISH: J4.7 (P7)
- new net CONTROL_1_GRN: D7.2 (K), J4.5 (P5)
- new net CONTROL_1_ORN: J4.3 (P3)
- new net CONTROL_1_RESET: J4.2 (P2)
- new net CONTROL_1_WHT: D2.1 (A), J4.9 (P9)
- new net CONTROL_1_YEL: J4.4 (P4)
- new net CONTROL_2_BLK_RED: J3.12 (P12)
- new net CONTROL_2_BLU: D8.2 (K), J3.6 (P6)
- new net CONTROL_2_BRN: J3.1 (P1)
- new net CONTROL_2_ENGLISH: J3.7 (P7)
- new net CONTROL_2_GRN: D5.2 (K), J3.5 (P5)
- new net CONTROL_2_ORN: J3.3 (P3)
- new net CONTROL_2_RESET: J3.2 (P2)
- new net CONTROL_2_WHT: D3.1 (A), J3.9 (P9)
- new net CONTROL_2_YEL: J3.4 (P4)
- new net GAME_CARD_27: C16.1, R16.2
- new net J15 - FLIP-FLOP/ENGLISH 703494-2/(1): D5.1 (A)
- new net J15 - FLIP-FLOP/ENGLISH 703494-2/(2): D7.1 (A)
- new net J15 - FLIP-FLOP/ENGLISH 703494-2/(7): D6.1 (A)
- new net J15 - FLIP-FLOP/ENGLISH 703494-2/(8): D8.1 (A)
- no-connect marks 21 -> 19
Other:
- note added: ".4 TO 5.4V"
- note added: "0V - OFF\n.6V - ON"
- note added: "1.27V\nWITH\nRESET\nCLOSED"
- note added: "A"
- note added: "C"
- note added: "CROWBAR\nRESET"
- note added: "G"
- note added: "HAND\nCONTROL\nNO.1"
- note added: "HAND\nCONTROL\nNO.2"
- note added: "RESET"
- note added: "TARGET"
- moved on the sheet: C17, C18, FB1, FB2, R54, S1, TP4

Commit message: terminei de transcrever a PCB toda. Deixei de fora de propósito o estágio de modulação RF do sinal. É pouca coisa, posso adicionar amanhã ou depois... Gerei também um PDFão
Parts:
- removed R?: 8.2k, symbol R
- added BATT1, JU1, JU11, JU3, JU4, JU5: JUMPER, symbol JUMPER
- added C13: .01, symbol CP1
- added C14, C15: 470 MFD 16V, symbol CAPAPOL
- added C2: 47 MFD 16V, symbol CAPAPOL
- added FB3: FERRITE, symbol FERRITE
- added J1: POWER_JACK, symbol JACK_2P
- added Q1: 142N9, symbol NPN
- added R45: 1.5k, symbol R
- added TP1: 5.6V, symbol TST
- added Z1: 6.2V, symbol ZENER
Connections:
- net CONTROL_1_BRN is gone; now on net +5.6V: J4.1 (P1)
- net CONTROL_2_BRN is gone; now on net +5.6V: J3.1 (P1)
- net CONTROL_2_ENGLISH is gone; now on net CONTROL_1_ENGLISH: J3.7 (P7)
- net CONTROL_2_YEL is gone; now on net CONTROL_1_YEL: J3.4 (P4)
- net GAME_CARD_34 is gone; now on net GAME_CARD_30: GAME_CARD_1.30 (P30), GAME_CARD_1.34 (P34), R2.1
- net GAME_CARD_42 is gone; now on net CONTROL_1_ENGLISH: GAME_CARD_1.42 (P42), R9.1
- net J6 - PLAYER NO.1 GEN 703493-2/(2) is gone; now on net CONTROL_1_VERT: C8.1
- net +5.6V: now also C13.1, C14.1, C15.1, FB3.1, JU4.1, Q1.1 (E), Q1.3 (C), R45.1, TP1.1
- net CONTROL_1_ORN: now also GAME_CARD_1.9 (P9)
- net CONTROL_1_RESET: now also JU1.1
- net CONTROL_1_YEL: now also GAME_CARD_1.38 (P38)
- net CONTROL_2_RESET: now also GAME_CARD_1.15 (P15), JU11.1
- net GAME_CARD_19: now also GAME_CARD_1.19 (P19)
- net GAME_CARD_23: now also GAME_CARD_1.23 (P23); no longer GAME_CARD_1.19 (P19)
- net GAME_CARD_27: now also GAME_CARD_1.27 (P27)
- net GND: now also BATT1.2, C13.2, C14.2, C15.2, C2.2, J1.3, Z1.1 (A)
- net GAME_CARD_13: now reaches GAME_CARD_1.13 (P13)
- net GAME_CARD_13: now also JU5.1
- net +9V: now reaches GAME_CARD_1.2 (P2), GAME_CARD_1.4 (P4)
- net +9V: now also J1.1
- net at GAME_CARD_1.3 (P3): now also C2.1
- net GAME_CARD_31: now reaches GAME_CARD_1.31 (P31), GAME_CARD_1.39 (P39)
- net GAME_CARD_31: now also JU3.1
- net GAME_CARD_35: now reaches GAME_CARD_1.35 (P35), GAME_CARD_1.37 (P37)
- net CONTROL_1_BLK_RED: no longer names the net of J4.12 (P12)
- net CONTROL_2_BLK_RED: no longer names the net of J3.12 (P12)
- net W3: no longer names the net of GAME_CARD_1.41 (P41)
- new net: Q1.2 (B), R45.2, Z1.2 (K)
- new net: BATT1.1, J1.2
- new net J11 - GATE MATRIX 703495-2/(1): JU1.2
- new net J11 - GATE MATRIX 703495-2/(10): JU11.2
- new net J11 - GATE MATRIX 703495-2/(3): JU3.2
- new net J11 - GATE MATRIX 703495-2/(6): JU4.2
- new net J11 - GATE MATRIX 703495-2/(8): JU5.2
- no-connect marks 19 -> 11
Other:
- note added: "(?!)"
- note added: "5.6V"
- note added: "MAGNAVOX ODYSSEY 1TL200BLAK SCHEMATIC DIAGRAM"
- note added: "REG\n+5.6V"
- note added: "Redrawn on KICAD by Felipe Corrêa da Silva Sanches <juca@members.fsf.org>"
- note added: "Scanned from original service manual by David WINTER"
- note added: "W3 (?!)"
- moved on the sheet: C1, C10, C11, C12, C16, C17, C18, C19, C20, C3, C4, C5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
