File: MagnavoxOdyssey1/MagnavoxOdyssey1.kicad_sch (KiCad schematic)
At the start: 99 parts, among them J101 Barrel_Jack_Switch, J20 CONN_6, J3 CONN_12, J4 CONN_12, Q1 142N9, Q2 142N9

Commit message: update to kicad 9
Parts:
- Q1, Q2: symbol Device:Q_NPN_EBC -> Transistor_BJT:Q_NPN_EBC
