File: MagnavoxOdyssey1/MagnavoxOdyssey1.kicad_sch (KiCad schematic)
At the start: 99 parts, among them J101 Barrel_Jack_Switch, J20 CONN_6, J3 CONN_12, J4 CONN_12, Q1 142N9, Q2 142N9

Commit message: npn model
Parts:
- R13: value 33k 5% -> 33k
- R19: value 130k 5% -> 130k
- R37: value R -> 0
Changed lines of the file:
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@@
 			)
 		)
-		(property "Value" "130k 5%"
+		(property "Value" "130k"
 			(at 652.0434 434.0352 0)
 			(effects
@@
 			)
 		)
-		(property "Value" "R"
+		(property "Value" "0"
 			(at 296.4434 748.9952 0)
 			(effects
@@
 			)
 		)
-		(property "Value" "33k 5%"
+		(property "Value" "33k"
 			(at 248.3866 406.0952 0)
 			(effects
@@
 			)
 		)
+		(property "Sim.Device" "NPN"
+			(at 474.98 269.24 0)
+			(effects
+				(font
+					(size 1.27 1.27)
+				)
+				(hide yes)
+			)
+		)
+		(property "Sim.Type" "VBIC"
+			(at 474.98 269.24 0)
+			(effects
+				(font
+					(size 1.27 1.27)
+				)
+				(hide yes)
+			)
+		)
+		(property "Sim.Pins" "1=E 2=B 3=C"
+			(at 474.98 269.24 0)
+			(effects
+				(font
+					(size 1.27 1.27)
+				)
+				(hide yes)
+			)
+		)
 		(pin "1"
 		)
@@
 			(at 629.92 238.76 0)
 			(effects
+				(font
+					(size 1.27 1.27)
+				)
+				(hide yes)
+			)
+		)
+		(property "Sim.Device" "NPN"
+			(at 629.92 238.76 0)
+			(effects
+				(font
+					(size 1.27 1.27)
+				)
+				(hide yes)
+			)
+		)
+		(property "Sim.Type" "VBIC"
+			(at 629.92 238.76 0)
+			(effects
+				(font
+					(size 1.27 1.27)
+				)
+				(hide yes)
+			)
+		)
+		(property "Sim.Pins" "1=E 2=B 3=C"
+			(at 629.92 238.76 0)
+			(effects
